Commit message: quadraped

File: body.urdf (robot description, URDF)
Before this commit: robot robot, 3 links, 2 joints
Links:
- added link LeftLeg, mass 1; collision box size=1 0.2 0.2; visual box size=1 0.2 0.2
- added link LowerBackLeg, mass 1; collision box size=0.2 0.2 1; visual box size=0.2 0.2 1
- added link LowerFrontLeg, mass 1; collision box size=0.2 0.2 1; visual box size=0.2 0.2 1
- added link LowerLeftLeg, mass 1; collision box size=0.2 0.2 1; visual box size=0.2 0.2 1
- added link LowerRightLeg, mass 1; collision box size=0.2 0.2 1; visual box size=0.2 0.2 1
- added link RightLeg, mass 1; collision box size=1 0.2 0.2; visual box size=1 0.2 0.2
- link BackLeg: geometry collision box size=0.2 1 0.2; visual box size=0.2 1 0.2
- link FrontLeg: geometry collision box size=0.2 1 0.2; visual box size=0.2 1 0.2
Joints:
- added joint BackLeg_LowerBackLeg: type revolute, parent BackLeg, child LowerBackLeg, origin xyz=0 -1 0 rpy=0 0 0, axis 1 0 0, limit lower=-3.14159 upper=3.14159 effort=0.0 velocity=0.0
- added joint FrontLeg_LowerFrontLeg: type revolute, parent FrontLeg, child LowerFrontLeg, origin xyz=0 1 0 rpy=0 0 0, axis 1 0 0, limit lower=-3.14159 upper=3.14159 effort=0.0 velocity=0.0
- added joint LeftLeg_LowerLeftLeg: type revolute, parent LeftLeg, child LowerLeftLeg, origin xyz=-1 0 0 rpy=0 0 0, axis 0 1 0, limit lower=-3.14159 upper=3.14159 effort=0.0 velocity=0.0
- added joint RightLeg_LowerRightLeg: type revolute, parent RightLeg, child LowerRightLeg, origin xyz=1 0 0 rpy=0 0 0, axis 0 1 0, limit lower=-3.14159 upper=3.14159 effort=0.0 velocity=0.0
- added joint Torso_LeftLeg: type revolute, parent Torso, child LeftLeg, origin xyz=-0.5 0 1 rpy=0 0 0, axis 0 1 0, limit lower=-3.14159 upper=3.14159 effort=0.0 velocity=0.0
- added joint Torso_RightLeg: type revolute, parent Torso, child RightLeg, origin xyz=0.5 0 1 rpy=0 0 0, axis 0 1 0, limit lower=-3.14159 upper=3.14159 effort=0.0 velocity=0.0
- joint Torso_BackLeg: axis 0 1 0 -> 1 0 0; origin xyz=1 0 1 rpy=0 0 0 -> xyz=0 -0.5 1 rpy=0 0 0
- joint Torso_FrontLeg: axis 0 1 0 -> 1 0 0; origin xyz=2 0 1 rpy=0 0 0 -> xyz=0 0.5 1 rpy=0 0 0

Commit message: final project dog

File: body.urdf (robot description, URDF)
Before this commit: robot robot, 9 links, 8 joints
Links:
- added link Head, mass 1; collision box size=0.5 0.5 0.5; visual box size=0.5 0.5 0.5
- added link Neck, mass 1; collision box size=0.2 0.2 1; visual box size=0.2 0.2 1
- link Torso: geometry collision box size=2 1 0.2; visual box size=2 1 0.2
Joints:
- added joint Neck_Head: type revolute, parent Neck, child Head, origin xyz=0 -1 0 rpy=0 0 0, axis 1 0 0, limit lower=-3.14159 upper=3.14159 effort=0.0 velocity=0.0
- added joint Torso_Neck: type revolute, parent Torso, child Neck, origin xyz=0 -0.5 1 rpy=0 0 0, axis 1 0 0, limit lower=-3.14159 upper=3.14159 effort=0.0 velocity=0.0

Commit message: snake draft

File: body.urdf (robot description, URDF)
Before this commit: robot robot, 11 links, 10 joints
Links:
- removed link BackLeg
- removed link FrontLeg
- removed link Head
- removed link LeftLeg
- removed link LowerBackLeg
- removed link LowerFrontLeg
- removed link LowerLeftLeg
- removed link LowerRightLeg
- removed link Neck
- removed link RightLeg
- removed link Torso
- added link Link0, mass 1; collision box size=1 1 2; visual box size=1 1 2
- added link Link1, mass 1; collision box size=3 1 1; visual box size=3 1 1
- added link Link2, mass 1; collision box size=1 2 2; visual box size=1 2 2
- added link Link3, mass 1; collision box size=2 2 2; visual box size=2 2 2
- added link Link4, mass 1; collision box size=3 1 2; visual box size=3 1 2
Joints:
- removed joint BackLeg_LowerBackLeg
- removed joint FrontLeg_LowerFrontLeg
- removed joint LeftLeg_LowerLeftLeg
- removed joint Neck_Head
- removed joint RightLeg_LowerRightLeg
- removed joint Torso_BackLeg
- removed joint Torso_FrontLeg
- removed joint Torso_LeftLeg
- removed joint Torso_Neck
- removed joint Torso_RightLeg
- added joint Link0_Link1: type revolute, parent Link0, child Link1, origin xyz=0 -0.5 0.5 rpy=0 0 0, axis 1 0 0, limit lower=-3.14159 upper=3.14159 effort=0.0 velocity=0.0
- added joint Link1_Link2: type revolute, parent Link1, child Link2, origin xyz=0 -1.0 0.5 rpy=0 0 0, axis 1 0 0, limit lower=-3.14159 upper=3.14159 effort=0.0 velocity=0.0
- added joint Link2_Link3: type revolute, parent Link2, child Link3, origin xyz=0 -2.0 0.5 rpy=0 0 0, axis 1 0 0, limit lower=-3.14159 upper=3.14159 effort=0.0 velocity=0.0
- added joint Link3_Link4: type revolute, parent Link3, child Link4, origin xyz=0 -2.0 0.5 rpy=0 0 0, axis 1 0 0, limit lower=-3.14159 upper=3.14159 effort=0.0 velocity=0.0

Commit message: a7

File: body.urdf (robot description, URDF)
Before this commit: robot robot, 8 links, 7 joints
Links:
- added link Link8, mass 1; collision box size=2.398309300143074 1.992692602563424 1.2064858505115161; visual box size=2.398309300143074 1.992692602563424 1.2064858505115161
- link Link0: geometry collision box size=1.0760013001368756 1.3568048230320717 1.3173941924292205; visual box size=1.0760013001368756 1.3568048230320717 1.3173941924292205
- link Link1: geometry collision box size=2.5544561164978483 1.309535217542901 1.2730478950417532; visual box size=2.5544561164978483 1.309535217542901 1.2730478950417532
- link Link2: geometry collision box size=1.6335094958753034 1.296324472086901 1.0649083689889434; visual box size=1.6335094958753034 1.296324472086901 1.0649083689889434
- link Link3: geometry collision box size=1.4212709960034706 1.0467287001329841 1.0648853820782502; visual box size=1.4212709960034706 1.0467287001329841 1.0648853820782502
- link Link4: geometry collision box size=1.222475955915839 1.0005554240335048 1.0300448775656683; visual box size=1.222475955915839 1.0005554240335048 1.0300448775656683
- link Link5: geometry collision box size=1.3171797837656745 1.1823950421400773 1.770918676037406; visual box size=1.3171797837656745 1.1823950421400773 1.770918676037406
- link Link6: geometry collision box size=2.771408834738364 1.5792750999044578 1.7567575866559006; visual box size=2.771408834738364 1.5792750999044578 1.7567575866559006
- link Link7: geometry collision box size=2.702040663571811 1.878733031131754 1.8992892755682478; visual box size=2.702040663571811 1.878733031131754 1.8992892755682478
Joints:
- added joint Link7_Link8: type revolute, parent Link7, child Link8, origin xyz=-1.385704417369182 -0.7896375499522289 0 rpy=0 0 0, axis 1 0 0, limit lower=-3.14159 upper=3.14159 effort=0.0 velocity=0.0
- joint Link0_Link1: origin xyz=0 -0.9664143691669067 0.5 rpy=0 0 0 -> xyz=0 -0.6784024115160359 0.5 rpy=0 0 0
- joint Link1_Link2: origin xyz=0 -1.2435786607889827 0.5 rpy=0 0 0 -> xyz=0.5380006500684378 0 0.6586970962146103 rpy=0 0 0
- joint Link2_Link3: axis 1 0 0 -> 0 1 0; origin xyz=0 -1.184684576719972 0.5 rpy=0 0 0 -> xyz=0 0.6547676087714505 0.6365239475208766 rpy=0 0 0
- joint Link3_Link4: origin xyz=0 -1.7447691161115126 0.5 rpy=0 0 0 -> xyz=0 -0.6481622360434505 -0.5324541844944717 rpy=0 0 0
- joint Link4_Link5: axis 1 0 0 -> 0 1 0; origin xyz=0 -1.7931310275475896 0.5 rpy=0 0 0 -> xyz=0 -0.5233643500664921 0.5324426910391251 rpy=0 0 0
- joint Link5_Link6: origin xyz=0 -1.3319069356865882 0.5 rpy=0 0 0 -> xyz=0.6112379779579195 -0.5002777120167524 0 rpy=0 0 0
- joint Link6_Link7: axis 1 0 0 -> 0 1 0; origin xyz=0 -1.38101488724173 0.5 rpy=0 0 0 -> xyz=-0.6585898918828372 0.5911975210700386 0 rpy=0 0 0

Commit message: edits to 3d

File: body.urdf (robot description, URDF)
Before this commit: robot robot, 9 links, 8 joints
Links:
- removed link Link4
- removed link Link5
- removed link Link6
- removed link Link7
- removed link Link8
- link Link0: geometry collision box size=1.4844361990662898 1.2729558655143256 1.7043476783825864; visual box size=1.4844361990662898 1.2729558655143256 1.7043476783825864
- link Link1: geometry collision box size=2.974268783640298 1.9519447543793165 1.5314842561006858; visual box size=2.974268783640298 1.9519447543793165 1.5314842561006858
- link Link2: geometry collision box size=2.697914819007628 1.798907563574574 1.4402109447852587; visual box size=2.697914819007628 1.798907563574574 1.4402109447852587
- link Link3: geometry collision box size=1.2269472500048724 1.6245799679212087 1.370606747873357; visual box size=1.2269472500048724 1.6245799679212087 1.370606747873357
Joints:
- removed joint Link3_Link4
- removed joint Link4_Link5
- removed joint Link5_Link6
- removed joint Link6_Link7
- removed joint Link7_Link8
- joint Link0_Link1: origin xyz=0 -0.6784024115160359 0.5 rpy=0 0 0 -> xyz=0 -0.6364779327571628 0.5 rpy=0 0 0
- joint Link1_Link2: origin xyz=0.5380006500684378 0 0.6586970962146103 rpy=0 0 0 -> xyz=0.7422180995331449 0 0.8521738391912932 rpy=0 0 0
- joint Link2_Link3: origin xyz=0 0.6547676087714505 0.6365239475208766 rpy=0 0 0 -> xyz=0 0.9759723771896582 0.7657421280503429 rpy=0 0 0

Commit message: a7

File: body.urdf (robot description, URDF)
Before this commit: robot robot, 4 links, 3 joints
Links:
- added link Link4, mass 1; collision box size=2.5003120024902814 1.1993978867513082 1.064744484839289; visual box size=2.5003120024902814 1.1993978867513082 1.064744484839289
- added link Link5, mass 1; collision box size=2.3623454399533816 1.259843202247656 1.9140976210862886; visual box size=2.3623454399533816 1.259843202247656 1.9140976210862886
- added link Link6, mass 1; collision box size=1.480254596298179 1.450743256439994 1.2908871022970492; visual box size=1.480254596298179 1.450743256439994 1.2908871022970492
- added link Link7, mass 1; collision box size=2.3870365416779458 1.8093292400459253 1.5785276689428382; visual box size=2.3870365416779458 1.8093292400459253 1.5785276689428382
- link Link0: geometry collision box size=1 1 2; visual box size=1 1 2
- link Link1: geometry collision box size=2.7917211168709373 1.0214955044217757 1.3194438183491368; visual box size=2.7917211168709373 1.0214955044217757 1.3194438183491368
- link Link2: geometry collision box size=1.0603956276910673 1.9722469762955868 1.5945174240440845; visual box size=1.0603956276910673 1.9722469762955868 1.5945174240440845
- link Link3: geometry collision box size=2.0341657763272387 1.7367572191940757 1.2658857967252641; visual box size=2.0341657763272387 1.7367572191940757 1.2658857967252641
Joints:
- added joint Link3_Link4: type revolute, parent Link3, child Link4, origin xyz=2.0341657763272387 0 0 rpy=0 0 0, axis 1 0 0, limit lower=-3.14159 upper=3.14159 effort=0.0 velocity=0.0
- added joint Link4_Link5: type revolute, parent Link4, child Link5, origin xyz=2.5003120024902814 0 0 rpy=0 0 0, axis 1 0 0, limit lower=-3.14159 upper=3.14159 effort=0.0 velocity=0.0
- added joint Link5_Link6: type revolute, parent Link5, child Link6, origin xyz=-0.06898328126844988 1.229620544499482 0 rpy=0 0 0, axis 0 1 0, limit lower=-3.14159 upper=3.14159 effort=0.0 velocity=0.0
- added joint Link6_Link7: type revolute, parent Link6, child Link7, origin xyz=-0.4410454218276013 0 1.6024923616916689 rpy=0 0 0, axis 0 1 0, limit lower=-3.14159 upper=3.14159 effort=0.0 velocity=0.0
- joint Link0_Link1: origin xyz=0 -0.6364779327571628 0.5 rpy=0 0 0 -> xyz=0.5 0 1.0 rpy=0 0 0
- joint Link1_Link2: axis 1 0 0 -> 0 1 0; origin xyz=0.7422180995331449 0 0.8521738391912932 rpy=0 0 0 -> xyz=0.8958605584354686 0 1.6597219091745683 rpy=0 0 0
- joint Link2_Link3: origin xyz=0 0.9759723771896582 0.7657421280503429 rpy=0 0 0 -> xyz=-0.865662744589935 0 1.4569806211966108 rpy=0 0 0

Commit message: adding gui line

File: body.urdf (robot description, URDF)
Before this commit: robot robot, 8 links, 7 joints
Links:
- removed link Link3
- removed link Link4
- removed link Link5
- removed link Link6
- removed link Link7
- link Link1: geometry collision box size=2.2884035930674353 1.25983620860358 1.8279627087434456; visual box size=2.2884035930674353 1.25983620860358 1.8279627087434456
- link Link2: geometry collision box size=2.5483132639448005 1.6727222072932015 1.6105914924022091; visual box size=2.5483132639448005 1.6727222072932015 1.6105914924022091
Joints:
- removed joint Link2_Link3
- removed joint Link3_Link4
- removed joint Link4_Link5
- removed joint Link5_Link6
- removed joint Link6_Link7
- joint Link1_Link2: origin xyz=0.8958605584354686 0 1.6597219091745683 rpy=0 0 0 -> xyz=0.6442017965337177 1.1299181043017898 0 rpy=0 0 0
