Commit message: trying to evolve

File: body4.urdf (robot description, URDF)
Before this commit: robot robot, 3 links, 2 joints
Links:
- link Link0: geometry collision box size=2 1 1; visual box size=2 1 1
- link Link1: geometry collision box size=1 2 2; visual box size=1 2 2
- link Link2: geometry collision box size=1 2 1; visual box size=1 2 1
Joints:
- joint Link0_Link1: axis 1 0 0 -> 0 1 0; origin xyz=0.5 0 1.0 rpy=0 0 0 -> xyz=0.5 1.0 0 rpy=0 0 0
- joint Link1_Link2: origin xyz=0.6442017965337177 1.1299181043017898 0 rpy=0 0 0 -> xyz=0.5 1.5 0 rpy=0 0 0
